File: DIY-Module_TB67H450FNG/DIY-Module_TB67H450FNG.kicad_pcb (KiCad board)
At the start: 2 copper layers, 16.3 x 19 mm, 6 parts, among them IC1 Motor_A, IC2 Motor_B, J1 Conn_01x07_Pin, J2 Conn_01x07_Pin

Commit message: Removed capacitors & update README.md
Parts:
- removed C2, C4: 100nF, Capacitor_SMD:C_0805_2012Metric_Pad1.18x1.45mm_HandSolder
