File: PCBWay-Module_TB67H450FNG/PCBWay-Module_TB67H450FNG.kicad_pcb (KiCad board)
At the start: 2 copper layers, 16.3 x 19 mm, 4 parts, among them IC1 Motor_A, IC2 Motor_B, J1 Conn_01x07_Pin, J2 Conn_01x07_Pin

Commit message: Added capacitors
Parts:
- added C1: 100, Capacitor_SMD:C_0805_2012Metric, F.Cu at (116.5, 115.6)
- added C2: 100, Capacitor_SMD:C_0805_2012Metric, F.Cu at (116.3, 107.8)
- added C3: 100, Capacitor_THT:C_Disc_D4.3mm_W1.9mm_P5.00mm, F.Cu at (114.8, 120.0)
Routing:
- net GND: vias 79 -> 73
- net /VM: vias 16 -> 13
