File: PCBWay-Module_TB67H450FNG/PCBWay-Module_TB67H450FNG.kicad_pcb (KiCad board)
At the start: 2 copper layers, 16.3 x 19 mm, 7 parts, among them IC1 Motor_A, IC2 Motor_B, J1 Conn_01x07_Pin, J2 Conn_01x07_Pin

Commit message: panels again
Parts:
- C1, C2: value 100 -> 100n
- C3: value 100 -> 100u
- moved C2 7.75 mm to (116.6, 115.6)
- moved C1 7.70 mm to (116.7, 107.9)
Connections:
- C1 pad 1: /IN_B1 -> /OUT_B1
- C1 pad 2: /IN_B2 -> /OUT_B2
- C2 pad 1: /IN_A1 -> /OUT_A1
- C2 pad 2: /IN_A2 -> /OUT_A2
Routing:
- net /OUT_B2: vias 5 -> 3
- net /OUT_B1: vias 5 -> 3
- net /OUT_A2: vias 5 -> 3
- net /OUT_A1: vias 5 -> 3
Changed lines of the file:
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@@
 	(footprint "Capacitor_SMD:C_0805_2012Metric"
 		(layer "F.Cu")
-		(at 116.35 107.85 90)
+		(at 116.6 115.6 90)
 		(descr "Capacitor SMD 0805 (2012 Metric), square (rectangular) end terminal, IPC_7351 nominal, (Body size source: IPC-SM-782 page 76, https://www.pcb-3d.com/wordpress/wp-content/uploads/ipc-sm-782a_amendment_1_and_2.pdf, https://docs.google.com/spreadsheets/d/1BsfQQcO9C6DZCsRaXUlFlo91Tg2WpOkGARC1WS5S8t0/edit?usp=sharing), generated with kicad-footprint-generator")
 		(tags "capacitor")
@@
 			)
 		)
-		(property "Value" "100"
+		(property "Value" "100n"
 			(at 0 1.68 90)
 			(layer "F.Fab")
@@
 			(layers "F.Cu" "F.Paste" "F.Mask")
 			(roundrect_rratio 0.25)
-			(net 9 "/IN_A1")
+			(net 2 "/OUT_A1")
 			(pintype "passive")
 		)
@@
 			(layers "F.Cu" "F.Paste" "F.Mask")
 			(roundrect_rratio 0.25)
-			(net 8 "/IN_A2")
+			(net 1 "/OUT_A2")
 			(pintype "passive")
 		)
@@
 			)
 		)
-		(property "Value" "100"
+		(property "Value" "100u"
 			(at 2.5 2.2 0)
 			(layer "F.Fab")
@@
 	(footprint "Capacitor_SMD:C_0805_2012Metric"
 		(layer "F.Cu")
-		(at 116.45 115.6 90)
+		(at 116.7 107.9 90)
 		(descr "Capacitor SMD 0805 (2012 Metric), square (rectangular) end terminal, IPC_7351 nominal, (Body size source: IPC-SM-782 page 76, https://www.pcb-3d.com/wordpress/wp-content/uploads/ipc-sm-782a_amendment_1_and_2.pdf, https://docs.google.com/spreadsheets/d/1BsfQQcO9C6DZCsRaXUlFlo91Tg2WpOkGARC1WS5S8t0/edit?usp=sharing), generated with kicad-footprint-generator")
 		(tags "capacitor")
@@
 			)
 		)
-		(property "Value" "100"
+		(property "Value" "100n"
 			(at 0 1.68 90)
 			(layer "F.Fab")
@@
 			(layers "F.Cu" "F.Paste" "F.Mask")
 			(roundrect_rratio 0.25)
-			(net 11 "/IN_B1")
+			(net 3 "/OUT_B1")
 			(pintype "passive")
 		)
@@
 			(layers "F.Cu" "F.Paste" "F.Mask")
 			(roundrect_rratio 0.25)
-			(net 10 "/IN_B2")
+			(net 4 "/OUT_B2")
 			(pintype "passive")
 		)
@@
 	)
 	(via
-		(at 117 115)
-		(size 0.65)
-		(drill 0.35)
-		(layers "F.Cu" "B.Cu")
-		(free yes)
-		(net 1)
-	)
-	(via
-		(at 115.75 115)
-		(size 0.65)
-		(drill 0.35)
-		(layers "F.Cu" "B.Cu")
-		(free yes)
-		(net 1)
-	)
-	(via
 		(at 115.75 113.75)
 		(size 0.65)
@@
 	)
 	(via
-		(at 117.1 116.25)
-		(size 0.65)
-		(drill 0.35)
-		(layers "F.Cu" "B.Cu")
-		(free yes)
-		(net 2)
-	)
-	(via
-		(at 115.85 116.25)
-		(size 0.65)
-		(drill 0.35)
-		(layers "F.Cu" "B.Cu")
-		(free yes)
-		(net 2)
-	)
-	(via
 		(at 113.54 116.59)
 		(size 0.65)
@@
 	)
 	(via
-		(at 115.8 108.6)
-		(size 0.65)
-		(drill 0.35)
-		(layers "F.Cu" "B.Cu")
-		(free yes)
-		(net 3)
-	)
-	(via
 		(at 115.8 109.85)
-		(size 0.65)
-		(drill 0.35)
-		(layers "F.Cu" "B.Cu")
-		(free yes)
-		(net 3)
-	)
-	(via
-		(at 117.05 108.6)
 		(size 0.65)
 		(drill 0.35)
@@
 	)
 	(via
-		(at 116.95 107.35)
-		(size 0.65)
-		(drill 0.35)
-		(layers "F.Cu" "B.Cu")
-		(free yes)
-		(net 4)
-	)
-	(via
 		(at 113.54 106.31)
 		(size 0.65)
@@
 		(size 0.65)
 		(drill 0.35)
-		(layers "F.Cu" "B.Cu")
-		(free yes)
-		(net 4)
-	)
-	(via
-		(at 115.7 107.35)
-		(size 0.65)
-		(drill 0.35)
