File: PCBWay-Module_TB67H450FNG/PCBWay-Module_TB67H450FNG.kicad_sch (KiCad schematic)
At the start: 4 parts, among them IC1 Motor_A, IC2 Motor_B, J1 Conn_01x07_Pin, J2 Conn_01x07_Pin

Commit message: Added capacitors
Parts:
- added C1, C2: 100, Capacitor_SMD:C_0805_2012Metric, symbol Device:C_Small
- added C3: 100, Capacitor_THT:C_Disc_D4.3mm_W1.9mm_P5.00mm, symbol Device:C_Small
Connections:
- net GND: now also C3.2
- net IN_A1: now also C2.1
- net IN_A2: now also C2.2
- net IN_B1: now also C1.1
- net IN_B2: now also C1.2
- net VM: now also C3.1

Commit message: Modified capacitors value
Parts:
- C1, C2: value 100 -> 100n
- C3: value 100 -> 100u
Changed lines of the file:
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@@
 			)
 		)
-		(property "Value" "100"
+		(property "Value" "100n"
 			(at 87.376 44.196 0)
 			(effects
@@
 			)
 		)
-		(property "Value" "100"
+		(property "Value" "100n"
 			(at 86.106 103.886 0)
 			(effects
@@
 			)
 		)
-		(property "Value" "100"
+		(property "Value" "100u"
 			(at 130.556 107.696 0)
 			(effects

Commit message: panels again
Connections:
- net IN_A1: no longer C2.1
- net IN_A2: no longer C2.2
- net IN_B1: no longer C1.1
- net IN_B2: no longer C1.2
- net OUT_A1: now also C2.1
- net OUT_A2: now also C2.2
- net OUT_B1: now also C1.1
- net OUT_B2: now also C1.2
Other:
- moved on the sheet: C1, C2
Changed lines of the file:
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@@
 	(generator_version "8.0")
 	(paper "A4")
+	(junction
+		(at 40.64 101.6)
+		(diameter 0)
+		(color 0 0 0 0)
+	)
+	(junction
+		(at 40.64 41.91)
+		(diameter 0)
+		(color 0 0 0 0)
+	)
+	(junction
+		(at 40.64 46.99)
+		(diameter 0)
+		(color 0 0 0 0)
+	)
+	(junction
+		(at 40.64 106.68)
+		(diameter 0)
+		(color 0 0 0 0)
+	)
 	(wire
 		(pts
@@
 	(wire
 		(pts
-			(xy 36.83 106.68) (xy 46.99 106.68)
+			(xy 40.64 106.68) (xy 46.99 106.68)
+		)
+		(stroke
+			(width 0)
+			(type default)
+		)
+	)
+	(wire
+		(pts
+			(xy 36.83 106.68) (xy 40.64 106.68)
 		)
 		(stroke
@@
 	(wire
 		(pts
+			(xy 40.64 101.6) (xy 46.99 101.6)
+		)
+		(stroke
+			(width 0)
+			(type default)
+		)
+	)
+	(wire
+		(pts
 			(xy 121.92 78.74) (xy 123.19 78.74)
 		)
@@
 	(wire
 		(pts
+			(xy 40.64 41.91) (xy 46.99 41.91)
+		)
+		(stroke
+			(width 0)
+			(type default)
+		)
+	)
+	(wire
+		(pts
 			(xy 120.65 58.42) (xy 123.19 58.42)
 		)
@@
 	(wire
 		(pts
-			(xy 36.83 46.99) (xy 46.99 46.99)
+			(xy 36.83 46.99) (xy 40.64 46.99)
 		)
 		(stroke
@@
 	(wire
 		(pts
-			(xy 36.83 41.91) (xy 46.99 41.91)
+			(xy 36.83 41.91) (xy 40.64 41.91)
 		)
 		(stroke
@@
 	(wire
 		(pts
+			(xy 40.64 46.99) (xy 46.99 46.99)
+		)
+		(stroke
+			(width 0)
+			(type default)
+		)
+	)
+	(wire
+		(pts
 			(xy 36.83 39.37) (xy 46.99 39.37)
 		)
@@
 	(wire
 		(pts
-			(xy 36.83 101.6) (xy 46.99 101.6)
+			(xy 36.83 101.6) (xy 40.64 101.6)
 		)
 		(stroke
@@
 		)
 	)
-	(label "IN_B1"
-		(at 83.82 100.33 180)
-		(fields_autoplaced yes)
-		(effects
-			(font
-				(size 1.27 1.27)
-			)
-			(justify right bottom)
-		)
-	)
 	(label "VM"
 		(at 128.27 104.14 180)
@@
 		)
 	)
-	(label "IN_A2"
-		(at 85.09 45.72 180)
-		(fields_autoplaced yes)
-		(effects
-			(font
-				(size 1.27 1.27)
-			)
-			(justify right bottom)
-		)
-	)
-	(label "IN_B2"
-		(at 83.82 105.41 180)
-		(fields_autoplaced yes)
-		(effects
-			(font
-				(size 1.27 1.27)
-			)
-			(justify right bottom)
-		)
-	)
 	(label "OUT_A1"
 		(at 121.92 78.74 180)
@@
 	(label "IN_A1"
 		(at 120.65 53.34 180)
-		(fields_autoplaced yes)
-		(effects
-			(font
-				(size 1.27 1.27)
-			)
-			(justify right bottom)
-		)
-	)
-	(label "IN_A1"
-		(at 85.09 40.64 180)
 		(fields_autoplaced yes)
 		(effects
@@
 	(symbol
 		(lib_id "Device:C_Small")
-		(at 85.09 43.18 0)
+		(at 40.64 44.45 0)
 		(unit 1)
 		(exclude_from_sim no)
@@
 		(dnp no)
 		(property "Reference" "C2"
-			(at 87.376 41.656 0)
+			(at 42.926 42.926 0)
 			(effects
 				(font
@@
 		)
 		(property "Value" "100n"
-			(at 87.376 44.196 0)
+			(at 42.926 45.466 0)
 			(effects
 				(font
@@
 		)
 		(property "Footprint" "Capacitor_SMD:C_0805_2012Metric"
-			(at 85.09 43.18 0)
+			(at 40.64 44.45 0)
 			(effects
 				(font
@@
 		)
 		(property "Datasheet" "~"
-			(at 85.09 43.18 0)
+			(at 40.64 44.45 0)
 			(effects
 				(font
@@
 		)
 		(property "Description" "Unpolarized capacitor, small symbol"
-			(at 85.09 43.18 0)
+			(at 40.64 44.45 0)
 			(effects
 				(font
@@
 	(symbol
 		(lib_id "Device:C_Small")
-		(at 83.82 102.87 0)
+		(at 40.64 104.14 0)
 		(unit 1)
 		(exclude_from_sim no)
@@
 		(dnp no)
 		(property "Reference" "C1"
-			(at 86.106 101.346 0)
+			(at 42.926 102.616 0)
 			(effects
 				(font
@@
 		)
 		(property "Value" "100n"
-			(at 86.106 103.886 0)
+			(at 42.926 105.156 0)
 			(effects
 				(font
@@
 		)
 		(property "Footprint" "Capacitor_SMD:C_0805_2012Metric"
-			(at 83.82 102.87 0)
+			(at 40.64 104.14 0)
 			(effects
 				(font
@@
 		)
 		(property "Datasheet" "~"
-			(at 83.82 102.87 0)
+			(at 40.64 104.14 0)
 			(effects
 				(font
@@
 		)
 		(property "Description" "Unpolarized capacitor, small symbol"
-			(at 83.82 102.87 0)
-			(effects
-				(font
+			(at 40.64 104.14 0)
+			(effects
+				(font
